Commit message: Updated Urdf

File: merlin_description/urdf/merlin.xacro (robot description, xacro)
@@ -8,7 +8,7 @@
 <link name="base_link">
   <inertial>
-    <origin rpy="0 0 0" xyz="0.0069422690555417796 1.1328659698873208e-16 0.15830248883091955"/>
-    <mass value="1290.6879375075011"/>
-    <inertia ixx="110.85266" ixy="0.0" ixz="-1.995437" iyy="112.361273" iyz="0.0" izz="143.593266"/>
+    <origin rpy="0 0 0" xyz="-5.307067970072318e-17 0.011280305091993278 0.17566675028184617"/>
+    <mass value="1377.5746329157873"/>
+    <inertia ixx="129.080457" ixy="-0.0" ixz="-0.0" iyy="126.261878" iyz="-4.078849" izz="151.45766"/>
   </inertial>
   <visual>
@@ -28,10 +28,10 @@
 <link name="Waist_1">
   <inertial>
-    <origin rpy="0 0 0" xyz="0.049382820138855435 -1.339727353549568e-09 0.2971243460783741"/>
+    <origin rpy="0 0 0" xyz="0.049382820138855435 -1.339727353549568e-09 0.2971243460783748"/>
     <mass value="812.9704335382083"/>
     <inertia ixx="28.634617" ixy="-1e-06" ixz="4.185208" iyy="41.522955" iyz="-0.0" izz="28.378178"/>
   </inertial>
   <visual>
-    <origin rpy="0 0 0" xyz="-0.0 -0.0 -0.762"/>
+    <origin rpy="0 0 0" xyz="-0.0 -0.0 -0.822325"/>
     <geometry>
       <mesh filename="package://merlin_description/meshes/Waist_1.stl" scale="0.001 0.001 0.001"/>
@@ -40,5 +40,5 @@
   </visual>
   <collision>
-    <origin rpy="0 0 0" xyz="-0.0 -0.0 -0.762"/>
+    <origin rpy="0 0 0" xyz="-0.0 -0.0 -0.822325"/>
     <geometry>
       <mesh filename="package://merlin_description/meshes/Waist_1.stl" scale="0.001 0.001 0.001"/>
@@ -48,10 +48,10 @@
 <link name="Shoulder_1">
   <inertial>
-    <origin rpy="0 0 0" xyz="0.0 -0.19144610574590126 0.008004317446370424"/>
-    <mass value="261.9268819351425"/>
-    <inertia ixx="18.724068" ixy="-0.0" ixz="0.0" iyy="17.838364" iyz="-4.08305" izz="3.735585"/>
+    <origin rpy="0 0 0" xyz="-1.0466970051982582e-16 -0.19144610574590126 0.008004317446370424"/>
+    <mass value="261.92688193514255"/>
+    <inertia ixx="18.724068" ixy="-0.0" ixz="-0.0" iyy="17.838364" iyz="-4.08305" izz="3.735585"/>
   </inertial>
   <visual>
-    <origin rpy="0 0 0" xyz="0.0 0.1778 -1.119907"/>
+    <origin rpy="0 0 0" xyz="0.0 0.1778 -1.180232"/>
     <geometry>
       <mesh filename="package://merlin_description/meshes/Shoulder_1.stl" scale="0.001 0.001 0.001"/>
@@ -60,5 +60,5 @@
   </visual>
   <collision>
-    <origin rpy="0 0 0" xyz="0.0 0.1778 -1.119907"/>
+    <origin rpy="0 0 0" xyz="0.0 0.1778 -1.180232"/>
     <geometry>
       <mesh filename="package://merlin_description/meshes/Shoulder_1.stl" scale="0.001 0.001 0.001"/>
@@ -68,10 +68,10 @@
 <link name="Lower_Head_1">
   <inertial>
-    <origin rpy="0 0 0" xyz="-0.03615717486675757 3.4416913763379853e-15 -1.364503258161065e-07"/>
-    <mass value="2.2131276746402757"/>
+    <origin rpy="0 0 0" xyz="-0.0361571748667579 3.3306690738754696e-15 -1.364503260381511e-07"/>
+    <mass value="2.2131276746402775"/>
     <inertia ixx="0.0067" ixy="-0.0" ixz="0.0" iyy="0.007083" iyz="0.0" izz="0.004151"/>
   </inertial>
   <visual>
-    <origin rpy="0 0 0" xyz="0.3556 0.3048 -0.678455"/>
+    <origin rpy="1.5708 0 0" xyz="0.3556 0.3048 -0.73878"/>
     <geometry>
       <mesh filename="package://merlin_description/meshes/Lower_Head_1.stl" scale="0.001 0.001 0.001"/>
@@ -80,5 +80,5 @@
   </visual>
   <collision>
-    <origin rpy="0 0 0" xyz="0.3556 0.3048 -0.678455"/>
+    <origin rpy="0 0 0" xyz="0.3556 0.3048 -0.73878"/>
     <geometry>
       <mesh filename="package://merlin_description/meshes/Lower_Head_1.stl" scale="0.001 0.001 0.001"/>
@@ -88,10 +88,10 @@
 <link name="Upper_Head_1">
   <inertial>
-    <origin rpy="0 0 0" xyz="-0.05560621831749479 4.440892098500626e-16 0.045845863549680343"/>
+    <origin rpy="0 0 0" xyz="-0.05560621831749479 3.885780586188048e-16 0.04584586354968023"/>
     <mass value="3.012798664762447"/>
-    <inertia ixx="0.004849" ixy="-0.0" ixz="-0.0" iyy="0.006079" iyz="0.0" izz="0.004733"/>
+    <inertia ixx="0.004849" ixy="0.0" ixz="-0.0" iyy="0.006079" iyz="-0.0" izz="0.004733"/>
   </inertial>
   <visual>
-    <origin rpy="0 0 0" xyz="0.437896 0.3048 -0.632609"/>
+    <origin rpy="0 0 0" xyz="0.437896 0.3048 -0.692934"/>
     <geometry>
       <mesh filename="package://merlin_description/meshes/Upper_Head_1.stl" scale="0.001 0.001 0.001"/>
@@ -100,5 +100,5 @@
   </visual>
   <collision>
-    <origin rpy="0 0 0" xyz="0.437896 0.3048 -0.632609"/>
+    <origin rpy="0 0 0" xyz="0.437896 0.3048 -0.692934"/>
     <geometry>
       <mesh filename="package://merlin_description/meshes/Upper_Head_1.stl" scale="0.001 0.001 0.001"/>
@@ -108,10 +108,10 @@
 <link name="Face_Plate_1">
   <inertial>
-    <origin rpy="0 0 0" xyz="-0.003937912465997062 5.551115123125783e-17 -1.3645034135922884e-07"/>
-    <mass value="0.47960575442808734"/>
-    <inertia ixx="0.000647" ixy="-0.0" ixz="0.0" iyy="0.000326" iyz="0.0" izz="0.000326"/>
+    <origin rpy="0 0 0" xyz="-0.003937912465997173 1.1102230246251565e-16 -1.3645034124820654e-07"/>
+    <mass value="0.47960575442808745"/>
+    <inertia ixx="0.000647" ixy="0.0" ixz="0.0" iyy="0.000326" iyz="0.0" izz="0.000326"/>
   </inertial>
   <visual>
-    <origin rpy="0 0 0" xyz="0.526796 0.3048 -0.678455"/>
+    <origin rpy="0 0 0" xyz="0.526796 0.3048 -0.73878"/>
     <geometry>
       <mesh filename="package://merlin_description/meshes/Face_Plate_1.stl" scale="0.001 0.001 0.001"/>
@@ -120,5 +120,5 @@
   </visual>
   <collision>
-    <origin rpy="0 0 0" xyz="0.526796 0.3048 -0.678455"/>
+    <origin rpy="0 0 0" xyz="0.526796 0.3048 -0.73878"/>
     <geometry>
       <mesh filename="package://merlin_description/meshes/Face_Plate_1.stl" scale="0.001 0.001 0.001"/>
@@ -128,10 +128,10 @@
 <link name="Elbow_1">
   <inertial>
-    <origin rpy="0 0 0" xyz="-0.024071311155488457 0.07620000000000005 -1.3645031959885756e-07"/>
-    <mass value="131.1743823904856"/>
+    <origin rpy="0 0 0" xyz="-0.02407131115548833 0.07619999999999999 -1.3645031959885756e-07"/>
+    <mass value="131.17438239048553"/>
     <inertia ixx="0.57509" ixy="-0.0" ixz="0.0" iyy="4.777681" iyz="-0.0" izz="4.709359"/>
   </inertial>
   <visual>
-    <origin rpy="0 0 0" xyz="-0.0 0.381 -0.678455"/>
+    <origin rpy="0 0 0" xyz="-0.0 0.381 -0.73878"/>
     <geometry>
       <mesh filename="package://merlin_description/meshes/Elbow_1.stl" scale="0.001 0.001 0.001"/>
@@ -140,5 +140,5 @@
   </visual>
   <collision>
-    <origin rpy="0 0 0" xyz="-0.0 0.381 -0.678455"/>
+    <origin rpy="0 0 0" xyz="-0.0 0.381 -0.73878"/>
     <geometry>
       <mesh filename="package://merlin_description/meshes/Elbow_1.stl" scale="0.001 0.001 0.001"/>
@@ -147,8 +147,8 @@
 </link>
 <joint name="waist" type="revolute">
-  <origin rpy="0 0 0" xyz="0.0 0.0 0.762"/>
+  <origin rpy="0 0 0" xyz="0.0 0.0 0.822325"/>
   <parent link="base_link"/>
   <child link="Waist_1"/>
-  <axis xyz="0.0 0.0 -1.0"/>
+  <axis xyz="0.0 0.0 1.0"/>
   <limit effort="100" lower="0.0" upper="5.061455" velocity="100"/>
 </joint>
@@ -163,5 +163,5 @@
   <parent link="Elbow_1"/>
   <child link="Lower_Head_1"/>
-  <axis xyz="1.0 0.0 -0.0"/>
+  <axis xyz="-1.0 0.0 -0.0"/>
 </joint>
 <joint name="wrist_flex" type="revolute">
@@ -184,7 +184,7 @@
   <axis xyz="0.0 1.0 0.0"/>
 </joint>
- <joint name="world" type="fixed">
-     <parent link="world_link"/>
-     <child link="base_link"/>
-   </joint>
+<joint name="world" type="fixed">
+  <parent link="world_link"/>
+  <child link="base_link"/>
+</joint>
 </robot>

Commit message: Sync

File: merlin_description/urdf/merlin.xacro (robot description, xacro)
@@ -73,5 +73,5 @@
   </inertial>
   <visual>
-    <origin rpy="1.5708 0 0" xyz="0.3556 0.3048 -0.73878"/>
+    <origin rpy="0 0 0" xyz="0.3556 0.3048 -0.73878"/>
     <geometry>
       <mesh filename="package://merlin_description/meshes/Lower_Head_1.stl" scale="0.001 0.001 0.001"/>
@@ -150,5 +150,5 @@
   <parent link="base_link"/>
   <child link="Waist_1"/>
-  <axis xyz="0.0 0.0 1.0"/>
+  <axis xyz="0.0 0.0 -1.0"/>
   <limit effort="100" lower="0.0" upper="5.061455" velocity="100"/>
 </joint>
@@ -182,5 +182,5 @@
   <parent link="Shoulder_1"/>
   <child link="Elbow_1"/>
-  <axis xyz="0.0 1.0 0.0"/>
+  <axis xyz="0.0 -1.0 0.0"/>
 </joint>
 <joint name="world" type="fixed">

Commit message: Sync

File: merlin_description/urdf/merlin.xacro (robot description, xacro)
@@ -169,5 +169,5 @@
   <parent link="Lower_Head_1"/>
   <child link="Upper_Head_1"/>
-  <axis xyz="-0.0 0.0 1.0"/>
+  <axis xyz="-0.0 0.0 -1.0"/>
   <limit effort="100" lower="-1.570796" upper="1.570796" velocity="100"/>
 </joint>
@@ -176,5 +176,5 @@
   <parent link="Upper_Head_1"/>
   <child link="Face_Plate_1"/>
-  <axis xyz="-1.0 0.0 0.0"/>
+  <axis xyz="1.0 0.0 0.0"/>
 </joint>
 <joint name="elbow" type="continuous">

Commit message: STL Updates

File: merlin_description/urdf/merlin.xacro (robot description, xacro)
@@ -73,5 +73,5 @@
   </inertial>
   <visual>
-    <origin rpy="1.5708 0 0" xyz="0.3556 0.3048 -0.73878"/>
+    <origin rpy="0 0 0" xyz="0.3556 0.3048 -0.73878"/>
     <geometry>
       <mesh filename="package://merlin_description/meshes/Lower_Head_1.stl" scale="0.001 0.001 0.001"/>
@@ -151,5 +151,5 @@
   <child link="Waist_1"/>
   <axis xyz="0.0 0.0 1.0"/>
-  <limit effort="100" lower="0.0" upper="5.061455" velocity="100"/>
+  <limit effort="100" lower="-4.537856" upper="0.523599" velocity="100"/>
 </joint>
 <joint name="shoulder" type="continuous">

Commit message: Added square cutting code

File: merlin_description/urdf/merlin.xacro (robot description, xacro)
@@ -150,11 +150,6 @@
   <parent link="base_link"/>
   <child link="Waist_1"/>
-<<<<<<< HEAD
-  <axis xyz="0.0 0.0 1.0"/>
+  <axis xyz="0.0 0.0 -1.0"/>
   <limit effort="100" lower="-4.537856" upper="0.523599" velocity="100"/>
-=======
-  <axis xyz="0.0 0.0 -1.0"/>
-  <limit effort="100" lower="0.0" upper="5.061455" velocity="100"/>
->>>>>>> b932141abf67f0c7553eb5c5d4d8cc8176031b3b
 </joint>
 <joint name="shoulder" type="continuous">
