Commit message: .

File: merlin_description/ros2_control/merlin.ros2_control.xacro (robot description, xacro)
@@ -98,5 +98,5 @@
     </xacro:macro>
 </robot>
-<!-- define lbr specific state interfaces as sensor, see
+<!-- define machine specific state interfaces as sensor, see
 https://github.com/ros-controls/roadmap/blob/master/design_drafts/components_architecture_and_urdf_examples.md -->
 <!-- <xacro:unless value="${sim}">

File: merlin_description/urdf/merlin/merlin.urdf.xacro (robot description, xacro)
@@ -2,5 +2,5 @@
 <!-- top level -->
 <robot name="merlin" xmlns:xacro="http://www.ros.org/wiki/xacro">
-    <!-- include the lbr med macro -->
+    <!-- include the merlin macro -->
     <xacro:include filename="$(find merlin_description)/urdf/merlin/merlin_description.urdf.xacro"/>
     <xacro:arg name="robot_name" default="merlin"/>

File: merlin_description/urdf/merlin/merlin_description.urdf.xacro (robot description, xacro)
@@ -26,5 +26,5 @@
         <origin rpy="0 0 0" xyz="0 0 0" />
         <geometry>
-          <mesh filename="package://merlin_description/meshes/merlin/base_link.stl"
+          <mesh filename="package://merlin_description/meshes/base_link.stl"
             scale="0.001 0.001 0.001" />
         </geometry>
@@ -34,5 +34,5 @@
         <origin rpy="0 0 0" xyz="0 0 0" />
         <geometry>
-          <mesh filename="package://merlin_description/meshes/merlin/base_link.stl"
+          <mesh filename="package://merlin_description/meshes/base_link.stl"
             scale="0.001 0.001 0.001" />
         </geometry>
@@ -49,5 +49,5 @@
         <origin rpy="0 0 0" xyz="-0.0 -0.0 -0.822325" />
         <geometry>
-          <mesh filename="package://merlin_description/meshes/merlin/Waist_1.stl"
+          <mesh filename="package://merlin_description/meshes/Waist_1.stl"
             scale="0.001 0.001 0.001" />
         </geometry>
@@ -57,5 +57,5 @@
         <origin rpy="0 0 0" xyz="-0.0 -0.0 -0.822325" />
         <geometry>
-          <mesh filename="package://merlin_description/meshes/merlin/Waist_1.stl"
+          <mesh filename="package://merlin_description/meshes/Waist_1.stl"
             scale="0.001 0.001 0.001" />
         </geometry>
@@ -78,5 +78,5 @@
         <origin rpy="0 0 0" xyz="0.0 0.1778 -1.180232" />
         <geometry>
-          <mesh filename="package://merlin_description/meshes/merlin/Shoulder_1.stl"
+          <mesh filename="package://merlin_description/meshes/Shoulder_1.stl"
             scale="0.001 0.001 0.001" />
         </geometry>
@@ -86,5 +86,5 @@
         <origin rpy="0 0 0" xyz="0.0 0.1778 -1.180232" />
         <geometry>
-          <mesh filename="package://merlin_description/meshes/merlin/Shoulder_1.stl"
+          <mesh filename="package://merlin_description/meshes/Shoulder_1.stl"
             scale="0.001 0.001 0.001" />
         </geometry>
@@ -106,5 +106,5 @@
         <origin rpy="0 0 0" xyz="0.3556 0.3048 -0.73878" />
         <geometry>
-          <mesh filename="package://merlin_description/meshes/merlin/Lower_Head_1.stl"
+          <mesh filename="package://merlin_description/meshes/Lower_Head_1.stl"
             scale="0.001 0.001 0.001" />
         </geometry>
@@ -114,5 +114,5 @@
         <origin rpy="0 0 0" xyz="0.3556 0.3048 -0.73878" />
         <geometry>
-          <mesh filename="package://merlin_description/meshes/merlin/Lower_Head_1.stl"
+          <mesh filename="package://merlin_description/meshes/Lower_Head_1.stl"
             scale="0.001 0.001 0.001" />
         </geometry>
@@ -134,5 +134,5 @@
         <origin rpy="0 0 0" xyz="0.437896 0.3048 -0.692934" />
         <geometry>
-          <mesh filename="package://merlin_description/meshes/merlin/Upper_Head_1.stl"
+          <mesh filename="package://merlin_description/meshes/Upper_Head_1.stl"
             scale="0.001 0.001 0.001" />
         </geometry>
@@ -142,5 +142,5 @@
         <origin rpy="0 0 0" xyz="0.437896 0.3048 -0.692934" />
         <geometry>
-          <mesh filename="package://merlin_description/meshes/merlin/Upper_Head_1.stl"
+          <mesh filename="package://merlin_description/meshes/Upper_Head_1.stl"
             scale="0.001 0.001 0.001" />
         </geometry>
@@ -164,5 +164,5 @@
         <origin rpy="0 0 0" xyz="0.526796 0.3048 -0.73878" />
         <geometry>
-          <mesh filename="package://merlin_description/meshes/merlin/Face_Plate_1.stl"
+          <mesh filename="package://merlin_description/meshes/Face_Plate_1.stl"
             scale="0.001 0.001 0.001" />
         </geometry>
@@ -172,5 +172,5 @@
         <origin rpy="0 0 0" xyz="0.526796 0.3048 -0.73878" />
         <geometry>
-          <mesh filename="package://merlin_description/meshes/merlin/Face_Plate_1.stl"
+          <mesh filename="package://merlin_description/meshes/Face_Plate_1.stl"
             scale="0.001 0.001 0.001" />
         </geometry>
@@ -192,5 +192,5 @@
         <origin rpy="0 0 0" xyz="-0.0 0.381 -0.73878" />
         <geometry>
-          <mesh filename="package://merlin_description/meshes/merlin/Elbow_1.stl"
+          <mesh filename="package://merlin_description/meshes/Elbow_1.stl"
             scale="0.001 0.001 0.001" />
         </geometry>
@@ -200,5 +200,5 @@
         <origin rpy="0 0 0" xyz="-0.0 0.381 -0.73878" />
         <geometry>
-          <mesh filename="package://merlin_description/meshes/merlin/Elbow_1.stl"
+          <mesh filename="package://merlin_description/meshes/Elbow_1.stl"
             scale="0.001 0.001 0.001" />
         </geometry>
