Commit message: Updated README

File: merlin_description/gazebo/merlin.gazebo.xacro (robot description, xacro)
@@ -1,10 +1,10 @@
 <?xml version="1.0" ?>
 <robot name="merlin" xmlns:xacro="http://www.ros.org/wiki/xacro" >
-  <xacro:macro name="merlin_gazebo" params="robot_name:=^|merlin">
+  <xacro:macro name="merlin_gazebo">
 <!-- ros_control-plugin -->
 <gazebo>
     <plugin name="gazebo_ros2_control" filename="libgazebo_ros2_control.so">
         <parameters>$(find merlin_bringup)/config/merlin_controllers.yml</parameters>
-        <robotNamespace>/${robot_name}</robotNamespace>
+        <robotNamespace>/merlin</robotNamespace>
     </plugin>
 </gazebo>

File: merlin_description/ros2_control/merlin.ros2_control.xacro (robot description, xacro)
@@ -1,5 +1,5 @@
 <robot xmlns:xacro="http://www.ros.org/wiki/xacro">
     <xacro:macro name="merlin_hardware_interface"
-        params="sim:=^|true remote_host:=^|INADDR_ANY port_id:=^|30200 robot_name:=^|merlin">
+        params="sim:=^|true remote_host:=^|INADDR_ANY port_id:=^|30200">
         <!-- arg for control mode -->
         <ros2_control name="merlin_hardware_interface" type="system">

Commit message: Need to upgrade to humble for pilz, ompl launches

File: merlin_description/gazebo/merlin.gazebo.xacro (robot description, xacro)
@@ -9,46 +9,38 @@
     </plugin>
 </gazebo>
-<gazebo reference="base_link">
+<gazebo reference="merlin_link_0">
   <material>Gazebo/Silver</material>
   <mu1>0.2</mu1>
   <mu2>0.2</mu2>
-  <selfCollide>true</selfCollide>
-  <gravity>true</gravity>
 </gazebo>
-<gazebo reference="Waist_1">
+<gazebo reference="merlin_link_1">
   <material>Gazebo/Red</material>
   <mu1>0.2</mu1>
   <mu2>0.2</mu2>
-  <selfCollide>true</selfCollide>
 </gazebo>
-<gazebo reference="Shoulder_1">
+<gazebo reference="merlin_link_2">
   <material>Gazebo/Red</material>
   <mu1>0.2</mu1>
   <mu2>0.2</mu2>
-  <selfCollide>true</selfCollide>
 </gazebo>
-<gazebo reference="Elbow_1">
+<gazebo reference="merlin_link_3">
   <material>Gazebo/Red</material>
   <mu1>0.2</mu1>
   <mu2>0.2</mu2>
-  <selfCollide>true</selfCollide>
 </gazebo>
-<gazebo reference="Lower_Head_1">
+<gazebo reference="merlin_link_4">
   <material>Gazebo/Silver</material>
   <mu1>0.2</mu1>
   <mu2>0.2</mu2>
-  <selfCollide>true</selfCollide>
 </gazebo>
-<gazebo reference="Upper_Head_1">
+<gazebo reference="merlin_link_5">
   <material>Gazebo/Silver</material>
   <mu1>0.2</mu1>
   <mu2>0.2</mu2>
-  <selfCollide>true</selfCollide>
 </gazebo>
-<gazebo reference="Face_Plate_1">
+<gazebo reference="merlin_link_6">
   <material>Gazebo/Black</material>
   <mu1>0.2</mu1>
   <mu2>0.2</mu2>
-  <selfCollide>true</selfCollide>
 </gazebo>
   </xacro:macro>

File: merlin_description/ros2_control/merlin.ros2_control.xacro (robot description, xacro)
@@ -1,8 +1,5 @@
 <robot xmlns:xacro="http://www.ros.org/wiki/xacro">
-    <xacro:macro name="merlin_hardware_interface"
-        params="sim:=^|true remote_host:=^|INADDR_ANY port_id:=^|30200">
-        <!-- arg for control mode -->
-        <ros2_control name="merlin_hardware_interface" type="system">
-            <!-- define hardware including parameters, also gazebo -->
+    <xacro:macro name="merlin_hardware_interface" params="sim:=^|true remote_host:=^|INADDR_ANY port_id:=^|30200">        <!-- arg for control mode -->
+        <ros2_control name="merlin_hardware_interface" type="system">            <!-- define hardware including parameters, also gazebo -->
             <xacro:if value="${sim}">
                 <hardware>
@@ -12,10 +9,10 @@
             <xacro:unless value="${sim}">
                 <hardware>
-                    <plugin>merlin_hwi/MerlinVelocityInterfaceHardware</plugin>
+                    <plugin>merlin_hardware_interface::MerlinHardwareInterface</plugin>
                     <param name="remote_host">${remote_host}</param>
                     <param name="port_id">${port_id}</param>
                 </hardware>
             </xacro:unless>
-            <joint name="waist">
+            <joint name="merlin_joint_0">
                 <command_interface name="velocity">
                     <param name="min">-1</param>
@@ -35,5 +32,5 @@
                 </xacro:unless>
             </joint>
-            <joint name="elbow">
+            <joint name="merlin_joint_1">
                 <command_interface name="velocity">
                     <param name="min">-1</param>
@@ -47,5 +44,5 @@
                 <state_interface name="position" />
             </joint>
-            <joint name="shoulder">
+            <joint name="merlin_joint_2">
                 <command_interface name="velocity">
                     <param name="min">-1</param>
@@ -59,5 +56,5 @@
                 <state_interface name="position" />
             </joint>
-            <joint name="wrist_rotation">
+            <joint name="merlin_joint_3">
                 <command_interface name="velocity">
                     <param name="min">-1</param>
@@ -71,5 +68,5 @@
                 <state_interface name="position" />
             </joint>
-            <joint name="wrist_flex">
+            <joint name="merlin_joint_4">
                 <command_interface name="velocity">
                     <param name="min">-1</param>
@@ -83,5 +80,5 @@
                 <state_interface name="position" />
             </joint>
-            <joint name="hand_roll">
+            <joint name="merlin_joint_5">
                 <command_interface name="velocity">
                     <param name="min">-1</param>
@@ -98,39 +95,2 @@
     </xacro:macro>
 </robot>
-<!-- define machine specific state interfaces as sensor, see
-https://github.com/ros-controls/roadmap/blob/master/design_drafts/components_architecture_and_urdf_examples.md -->
-<!-- <xacro:unless value="${sim}">
-                <sensor name="${robot_name}_fri_sensor">
-                    <state_interface name="sample_time"/>
-                    <state_interface name="session_state"/>
-                    <state_interface name="connection_quality"/>
-                    <state_interface name="safety_state"/>
-                    <state_interface name="operation_mode"/>
-                    <state_interface name="drive_state"/>
-                    <state_interface name="client_command_mode"/>
-                    <state_interface name="overlay_type"/>
-                    <state_interface name="control_mode"/>
-                    <state_interface name="time_stamp_sec"/>
-                    <state_interface name="time_stamp_nano_sec"/>
-                    <state_interface name="tracking_performance"/>
-                </sensor>
-            </xacro:unless> -->
-<!-- <joint name="${robot_name}_joint_6">
-<command_interface name="position">
-    <param name="min">-1</param>
-    <param name="max"> 1</param>
-</command_interface>
-<command_interface name="effort">
-    <param name="min">-1</param>
-    <param name="max"> 1</param>
-</command_interface>
-<state_interface name="position"/>
-<state_interface name="velocity"/>
-<state_interface name="effort"/>
-<xacro:unless value="${sim}">
-    <state_interface name="commanded_joint_position"/>
-    <state_interface name="commanded_torque"/>
-    <state_interface name="external_torque"/>
-    <state_interface name="ipo_joint_position"/>
-</xacro:unless>
-</joint> -->

File: merlin_description/urdf/merlin/merlin.urdf.xacro (robot description, xacro)
@@ -4,9 +4,8 @@
     <!-- include the merlin macro -->
     <xacro:include filename="$(find merlin_description)/urdf/merlin/merlin_description.urdf.xacro"/>
-    <xacro:arg name="robot_name" default="merlin"/>
     <xacro:arg name="sim" default="true"/>
     <!-- fix to world -->
     <link name="world"/>
     <!-- merlin -->
-    <xacro:merlin parent="world" robot_name="$(arg robot_name)" sim="$(arg sim)"/>
+    <xacro:merlin parent="world" sim="$(arg sim)"/>
 </robot>
