Commit message: Added Drill to urdf

File: merlin_description/urdf/merlin/merlin.urdf.xacro (robot description, xacro)
@@ -3,9 +3,24 @@
 <robot name="merlin" xmlns:xacro="http://www.ros.org/wiki/xacro">
     <!-- include the merlin macro -->
-    <xacro:include filename="$(find merlin_description)/urdf/merlin/merlin_description.urdf.xacro"/>
-    <xacro:arg name="sim" default="true"/>
+    <xacro:include filename="$(find merlin_description)/urdf/merlin/merlin_description.urdf.xacro" />
+    <xacro:include filename="$(find merlin_description)/urdf/turntable/turntable.urdf.xacro" />
+    <xacro:include filename="$(find merlin_description)/urdf/materials.urdf.xacro" />
+    <xacro:arg name="sim" default="true" />
+    <xacro:arg name="table" default="true" />
+    <xacro:arg name="tool" default="true" />
     <!-- fix to world -->
-    <link name="world"/>
+    <link name="world" />
     <!-- merlin -->
-    <xacro:merlin parent="world" sim="$(arg sim)"/>
+    <xacro:merlin parent="world" sim="$(arg sim)" />
+    <xacro:if value="$(arg table)">
+        <xacro:turntable parent="merlin_link_0" sim="$(arg sim)" />
+    </xacro:if>
+    <xacro:unless value="false">
+        <xacro:include filename="$(find merlin_description)/urdf/tools/basic_drill.urdf.xacro" />
+        <joint name="merlin_tool_joint" type="fixed">
+            <origin rpy="0 0 0" xyz="-0.008015 0.0 0.0" />
+            <parent link="merlin_link_6" />
+            <child link="tool_link_0" />
+        </joint>
+    </xacro:unless>
 </robot>

File: merlin_description/urdf/merlin/merlin_description.urdf.xacro (robot description, xacro)
@@ -7,5 +7,4 @@
     <xacro:property name="max_effort" value="300" />
     <xacro:property name="max_velocity" value="10" />
-    <xacro:include filename="$(find merlin_description)/urdf/materials.urdf.xacro" />
     <xacro:include filename="$(find merlin_description)/gazebo/merlin.gazebo.xacro" />
     <xacro:include filename="$(find merlin_description)/ros2_control/merlin.ros2_control.xacro" />
@@ -25,5 +24,5 @@
                 <origin rpy="0 0 0" xyz="0 0 0" />
                 <geometry>
-                    <mesh filename="package://merlin_description/meshes/link_0.stl" scale="0.001 0.001 0.001" />
+                    <mesh filename="package://merlin_description/meshes/merlin/link_0.stl" scale="0.001 0.001 0.001" />
                 </geometry>
                 <material name="silver" />
@@ -32,5 +31,5 @@
                 <origin rpy="0 0 0" xyz="0 0 0" />
                 <geometry>
-                    <mesh filename="package://merlin_description/meshes/link_0.stl" scale="0.001 0.001 0.001" />
+                    <mesh filename="package://merlin_description/meshes/merlin/link_0.stl" scale="0.001 0.001 0.001" />
                 </geometry>
             </collision>
@@ -52,5 +51,5 @@
                 <origin rpy="0 0 0" xyz="-0.0 -0.0 -0.822325" />
                 <geometry>
-                    <mesh filename="package://merlin_description/meshes/link_1.stl" scale="0.001 0.001 0.001" />
+                    <mesh filename="package://merlin_description/meshes/merlin/link_1.stl" scale="0.001 0.001 0.001" />
                 </geometry>
                 <material name="silver" />
@@ -59,5 +58,5 @@
                 <origin rpy="0 0 0" xyz="-0.0 -0.0 -0.822325" />
                 <geometry>
-                    <mesh filename="package://merlin_description/meshes/link_1.stl" scale="0.001 0.001 0.001" />
+                    <mesh filename="package://merlin_description/meshes/merlin/link_1.stl" scale="0.001 0.001 0.001" />
                 </geometry>
             </collision>
@@ -78,5 +77,5 @@
                 <origin rpy="0 0 0" xyz="0.0 0.1778 -1.180232" />
                 <geometry>
-                    <mesh filename="package://merlin_description/meshes/link_2.stl" scale="0.001 0.001 0.001" />
+                    <mesh filename="package://merlin_description/meshes/merlin/link_2.stl" scale="0.001 0.001 0.001" />
                 </geometry>
                 <material name="silver" />
@@ -85,5 +84,5 @@
                 <origin rpy="0 0 0" xyz="0.0 0.1778 -1.180232" />
                 <geometry>
-                    <mesh filename="package://merlin_description/meshes/link_2.stl" scale="0.001 0.001 0.001" />
+                    <mesh filename="package://merlin_description/meshes/merlin/link_2.stl" scale="0.001 0.001 0.001" />
                 </geometry>
             </collision>
@@ -104,5 +103,5 @@
                 <origin rpy="0 0 0" xyz="-0.0 0.381 -0.73878" />
                 <geometry>
-                    <mesh filename="package://merlin_description/meshes/link_3.stl" scale="0.001 0.001 0.001" />
+                    <mesh filename="package://merlin_description/meshes/merlin/link_3.stl" scale="0.001 0.001 0.001" />
                 </geometry>
                 <material name="silver" />
@@ -111,5 +110,5 @@
                 <origin rpy="0 0 0" xyz="-0.0 0.381 -0.73878" />
                 <geometry>
-                    <mesh filename="package://merlin_description/meshes/link_3.stl" scale="0.001 0.001 0.001" />
+                    <mesh filename="package://merlin_description/meshes/merlin/link_3.stl" scale="0.001 0.001 0.001" />
                 </geometry>
             </collision>
@@ -130,5 +129,5 @@
                 <origin rpy="0 0 0" xyz="0.3556 0.3048 -0.73878" />
                 <geometry>
-                    <mesh filename="package://merlin_description/meshes/link_4.stl" scale="0.001 0.001 0.001" />
+                    <mesh filename="package://merlin_description/meshes/merlin/link_4.stl" scale="0.001 0.001 0.001" />
                 </geometry>
                 <material name="silver" />
@@ -137,5 +136,5 @@
                 <origin rpy="0 0 0" xyz="0.3556 0.3048 -0.73878" />
                 <geometry>
-                    <mesh filename="package://merlin_description/meshes/link_4.stl" scale="0.001 0.001 0.001" />
+                    <mesh filename="package://merlin_description/meshes/merlin/link_4.stl" scale="0.001 0.001 0.001" />
                 </geometry>
             </collision>
@@ -157,5 +156,5 @@
                 <origin rpy="0 0 0" xyz="0.437896 0.3048 -0.692934" />
                 <geometry>
-                    <mesh filename="package://merlin_description/meshes/link_5.stl" scale="0.001 0.001 0.001" />
+                    <mesh filename="package://merlin_description/meshes/merlin/link_5.stl" scale="0.001 0.001 0.001" />
                 </geometry>
                 <material name="silver" />
@@ -164,5 +163,5 @@
                 <origin rpy="0 0 0" xyz="0.437896 0.3048 -0.692934" />
                 <geometry>
-                    <mesh filename="package://merlin_description/meshes/link_5.stl" scale="0.001 0.001 0.001" />
+                    <mesh filename="package://merlin_description/meshes/merlin/link_5.stl" scale="0.001 0.001 0.001" />
                 </geometry>
             </collision>
@@ -183,5 +182,5 @@
                 <origin rpy="0 0 0" xyz="0.526796 0.3048 -0.73878" />
                 <geometry>
-                    <mesh filename="package://merlin_description/meshes/link_6.stl" scale="0.001 0.001 0.001" />
+                    <mesh filename="package://merlin_description/meshes/merlin/link_6.stl" scale="0.001 0.001 0.001" />
                 </geometry>
                 <material name="silver" />
@@ -190,9 +189,8 @@
                 <origin rpy="0 0 0" xyz="0.526796 0.3048 -0.73878" />
                 <geometry>
-                    <mesh filename="package://merlin_description/meshes/link_6.stl" scale="0.001 0.001 0.001" />
+                    <mesh filename="package://merlin_description/meshes/merlin/link_6.stl" scale="0.001 0.001 0.001" />
                 </geometry>
             </collision>
         </link>
- <static>1</static>
         <xacro:merlin_gazebo />
         <!-- TODO: move modes to args, decouple urdf/gazebo/controls -->
